File: hardware/KiCad/ESC_v1.0/ESC_v1.0.kicad_sch (KiCad schematic)
At the start: 0 parts

Commit message: Update Kicad
Parts:
- added C1, C2, C3, C5: 100n, Capacitor_SMD:C_0402_1005Metric, symbol ESC-SchemSymLib:CL05B104KO5NNNC
- added C4: 4.7u, Capacitor_SMD:C_0402_1005Metric, symbol Device:C
- added C6, C8: 1u, Capacitor_SMD:C_0402_1005Metric, symbol Device:C
- added C7: 10n, Capacitor_SMD:C_0402_1005Metric, symbol Device:C
- added U1: STM32G484CEU6, Package_DFN_QFN:QFN-48-1EP_7x7mm_P0.5mm_EP5.6x5.6mm_ThermalVias, symbol ESC-SchemSymLib:STM32G484CEU6
Connections:
- new net +3V3: C1.1, C2.1, C3.1, C4.1, U1.1 (VBAT), U1.23 (VDD), U1.35 (VDD), U1.48 (VDD)
- new net +3V3A: C5.1, C6.1, C7.1, C8.1, U1.20 (VREF+), U1.21 (VDDA)
- new net GND: C1.2, C2.2, C3.2, C4.2, C5.2, C6.2, C7.2, C8.2, U1.PAD (VSS)
Other:
- company: (none) -> Bare Metal Foundry
- title: (none) -> Kururugi-ESC
