File: hardware/KiCad/ESC_v1.0/ESC_v1.0.kicad_sch (KiCad schematic)
At the start: 9 parts, among them U1 STM32G484CEU6

Commit message: Update on kicad
Parts:
- removed C4: 4.7u, Capacitor_SMD:C_0402_1005Metric, symbol Device:C
- removed C6, C8: 1u, Capacitor_SMD:C_0402_1005Metric, symbol Device:C
- removed C7: 10n, Capacitor_SMD:C_0402_1005Metric, symbol Device:C
- added C10, C11: 10p, Capacitor_SMD:C_0402_1005Metric, symbol ESC-SchemSymLib:CL05C100JB5NNNC
- added C13, C14, C15: C, symbol Device:C
- added C16, C6, C8: 1u, Capacitor_SMD:C_0603_1608Metric, symbol ESC-SchemSymLib:CL10A105KB8NNNC
- added C4: 4.7u, Capacitor_SMD:C_0805_2012Metric, symbol ESC-SchemSymLib:CL21A475KAQNNNE
- added C43: 1u, Capacitor_SMD:C_0402_1005Metric, symbol Device:C
- added C44: 100n, Capacitor_SMD:C_0402_1005Metric, symbol Device:C
- added C7: 10n, Capacitor_SMD:C_0402_1005Metric, symbol ESC-SchemSymLib:CL05B103KB5NNNC
- added C9: 100n, Capacitor_SMD:C_0402_1005Metric, symbol ESC-SchemSymLib:CL05B104KO5NNNC
- added D6: USB_LED, LED_SMD:LED_0603_1608Metric, symbol Device:LED
- added F1: MF-MSMF050-2, Resistor_SMD:R_1812_4532Metric, symbol Device:Polyfuse
- added J3: USB4105-GF-A, FC-FootprintLib:GCT_USB4105-GF-A, symbol FC-SchemSymbolLib:USB4105-GF-A
- added J4: Conn_ARM_SWD_TagConnect_TC2030-NL, Connector:Tag-Connect_TC2030-IDC-NL_2x03_P1.27mm_Vertical, symbol Connector:Conn_ARM_SWD_TagConnect_TC2030-NL
- added L1: L, symbol Device:L
- added R1, R32: 82k, Resistor_SMD:R_0402_1005Metric, symbol Device:R
- added R2, R3, R4, R5, R6: R, symbol Device:R
- added R31: 43k, Resistor_SMD:R_0402_1005Metric, symbol Device:R
- added R33: 250, Resistor_SMD:R_0402_1005Metric, symbol Device:R
- added R34, R35: 5.1k, Resistor_SMD:R_0402_1005Metric, symbol Device:R
- added TP1: ResetPad, symbol Connector:TestPoint
- added TP4: TestPoint Pad, TestPoint:TestPoint_Pad_D1.0mm, symbol Connector:TestPoint
- added U2: LM5160A, symbol ESC-SchemSymLib:LM5160ADNTR
- added U8: USBLC6-2SC6, Package_TO_SOT_SMD:SOT-23-6, symbol FC-SchemSymbolLib:USBLC6-2SC6
- added X1: 16MHz, Crystal:Crystal_SMD_2520-4Pin_2.5x2.0mm, symbol ESC-SchemSymLib:Crystal_GND24
- C1, C2, C3, C5: Distributor Link 1 https://www.digikey.com.au/en/products/detail/samsung-elect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 -> https://au.mouser.com/ProductDetail/Samsung-Electro-Mechani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; Distributor Link 2 https://au.mouser.com/ProductDetail/Samsung-Electro-Mechani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 -> https://www.digikey.com.au/en/products/detail/samsung-elect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
Connections:
- net +3V3: now also C4.1
- net +3V3A: now also C6.1, C7.1; no longer C5.1, U1.20 (VREF+)
- net DEBUG_SWDIO: now reaches U1.13 (PA5)
- net DEBUG_SWDIO: now also J4.2 (SWDIO)
- net DEBUG_SWCLK: now reaches U1.14 (PA6)
- net DEBUG_SWCLK: now also J4.4 (SWCLK)
- net DEBUG_SWO: now reaches U1.41 (PB3)
- net DEBUG_SWO: now also J4.6 (SWO)
- net BOOT0: now reaches U1.46 (PB8-BOOT0)
- net BOOT0: now also R1.2, TP1.1
- net HSE_IN: now reaches U1.5 (PF0-OSC_IN)
- net HSE_IN: now also C11.1, X1.3
- net HSE_OUT: now reaches U1.6 (PF1-OSC_OUT)
- net HSE_OUT: now also C10.1, X1.1
- net DEBUG_NRST: now reaches U1.7 (PG10-NRST)
- net DEBUG_NRST: now also C9.1, J4.3 (~{RESET})
- net GND renamed AGND
- net AGND: now also C10.2, C11.2, C14.2, C15.2, C16.2, C4.2, C43.2, C44.2, C6.2, C7.2, C8.2, C9.2, D6.1 (K), J3.A1 (GND), J3.B1 (GND), J3.SH1 (SHIELD), J3.SH2 (SHIELD), J3.SH3 (SHIELD), J3.SH4 (SHIELD), J4.5 (GND), R1.1, R32.1, R34.1, R35.1, R4.2, R6.1, U2.1 (AGND), U2.2 (PGND), U2.PAD (AGND), U8.2 (GND), X1.2, X1.4
- new net: D6.2 (A), R33.1
- new net: F1.1, J3.A4 (VBUS), J3.B4 (VBUS), U8.5 (VBUS)
- new net: C13.2, U2.10 (BST)
- new net: C13.1, L1.1, U2.11 (SW), U2.12 (SW)
- new net: R3.2, R4.1, U2.4 (EN/UVLO)
- new net: R2.2, U2.5 (RON)
- new net: C16.1, U2.6 (SS)
- new net: C14.1, U2.7 (FPWM), U2.9 (VCC)
- new net: R5.1, R6.2, U2.8 (FB)
- new net: J3.B5 (CC2), R35.2
- new net: J3.A5 (CC1), R34.2
- new net +10V: L1.2, R5.2
- new net +3.3V: J4.1 (VCC)
- new net +3V3REF: C5.1, C8.1, U1.20 (VREF+)
- new net USB_D+: J3.A6 (D1+), J3.B6 (D2+), U8.1 (I/O1), U8.6 (I/O1)
- new net USB_D-: J3.A7 (D1-), J3.B7 (D2-), U8.3 (I/O2), U8.4 (I/O2)
- new net USB_VBUS_SENSE: R31.1, R32.2
- new net VBAT: C15.1, R2.1, R3.1, U2.3 (VIN)
- new net VBUS: C43.1, C44.1, F1.2, R31.2, R33.2, TP4.1
- no-connect marks 0 -> 2
Other:
- note added: "CC1 and CC2 pulled down with 5.1k resistors => advertise USB devide mode --------- SBU1/2 for alternate DisplayPort mode --------- VBUS Sensing disabled"
- note added: "C_L1 = C_L2 = 2*(C_L - C_p) Assume stray capacitance C_p = 4pF R_EXT = 1/(2piFC_L2) !!!!!!!!!"
- note added: "Crystal Oscillator"
- note added: "DEBUG Tag Connect"
- note added: "General: Here we set OUT=(1A,10V), VIN=[4S, 6S]=[12, 60]V (ripple) --------------- Switching: FSW = min(FSW_max@VIN_min, FSW_max@VIN_max) = 981kHz RON = VOUT/FSW*10^10 = 110kR (TON=458ns) COT type BUCK: SW node high for TON if FB<REF. --------------- Inductor: L=VOx(VIN_max-VO)/(VIN_max*FSW*IO_max*0.4)=18µH. --------------- Other: Soft Start: CSS=1µF => TSS=200ms. Feedback: 10V to 2V => RFB2/RFB1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"
- note added: "I_limit = 500/R_ILIM Here we set I_limit = 2A --------------- Sitching logic: VSNS = V_IN1 * R7/(R6+R7) if VSNS > 0.8V => OUT = IN1 otherwise take the highest input --------------- We want: if V_IN1 > 5V => OUT = IN1"
- note added: "Internal NRESET Pullup resistor already included in the MCU"
- note added: "USB-C"
- moved on the sheet: C1, C2, C3, C5, U1
